Commit message: docker file removed, updated Readme

File: src/khm_description/urdf/khm_description copy.urdf (robot description, URDF)
Before this commit: robot khm_description, 28 links, 27 joints
Links:
- removed link imu_wheel_lb_link
- removed link imu_wheel_lf_link
- removed link imu_wheel_lm_link
- removed link imu_wheel_rb_link
- removed link imu_wheel_rf_link
- removed link imu_wheel_rm_link
- removed link wheel_lb_local
- removed link wheel_lf_local
- removed link wheel_lm_local
- removed link wheel_rb_local
- removed link wheel_rf_local
- removed link wheel_rm_local
- added link back_imu_rocker_left
- added link back_imu_rocker_right
- added link front_imu_rocker_left
- added link front_imu_rocker_right
- added link wheel_lf_thermal_frame
- link wheel_lb: geometry collision mesh filename=package://khm_description/meshes/wheel_lb_col.STL scale=1 1 1; visual mesh filename=package://khm_description/meshes/wheel_lb.dae scale=1 1 1
- link wheel_lf: geometry collision mesh filename=package://khm_description/meshes/wheel_lf_col.STL scale=1 1 1; visual mesh filename=package://khm_description/meshes/wheel_lf.dae scale=1 1 1
- link wheel_lm: geometry collision mesh filename=package://khm_description/meshes/wheel_lm_col.STL scale=1 1 1; visual mesh filename=package://khm_description/meshes/wheel_lm.dae scale=1 1 1
- link wheel_rb: geometry collision mesh filename=package://khm_description/meshes/wheel_rb_col.STL scale=1 1 1; visual mesh filename=package://khm_description/meshes/wheel_rb.dae scale=1 1 1
- link wheel_rf: geometry collision mesh filename=package://khm_description/meshes/wheel_rf_col.STL scale=1 1 1; visual mesh filename=package://khm_description/meshes/wheel_rf.dae scale=1 1 1
- link wheel_rm: geometry collision mesh filename=package://khm_description/meshes/wheel_rm_col.STL scale=1 1 1; visual mesh filename=package://khm_description/meshes/wheel_rm.dae scale=1 1 1
Joints:
- removed joint bogie_left_wheel_lm_local
- removed joint bogie_right_wheel_rm_local
- removed joint corner_lb_wheel_lb_local
- removed joint corner_lf_wheel_lf_local
- removed joint corner_rb_wheel_rb_local
- removed joint corner_rf_wheel_rf_local
- removed joint imu_wheel_lb_joint
- removed joint imu_wheel_lf_joint
- removed joint imu_wheel_lm_joint
- removed joint imu_wheel_rb_joint
- removed joint imu_wheel_rf_joint
- removed joint imu_wheel_rm_joint
- added joint corner_lf_wheel_lf_thermal_frame: type fixed, parent corner_lf, child wheel_lf_thermal_frame, origin xyz=0.0 0.0 0.0 rpy=1.575 0.000 3.067
- added joint rocker_left_back_imu: type fixed, parent rocker_left, child back_imu_rocker_left, origin xyz=0 0 0.2 rpy=0 1.507 0
- added joint rocker_left_front_imu: type fixed, parent rocker_left, child front_imu_rocker_left, origin xyz=0 0 0 rpy=0 1.507 0
- added joint rocker_right_back_imu: type fixed, parent rocker_right, child back_imu_rocker_right, origin xyz=0.2 0 0 rpy=0 3.14 0
- added joint rocker_right_front_imu: type fixed, parent rocker_right, child front_imu_rocker_right, origin xyz=0 0 0 rpy=0 3.14 0
- joint body_rocker_left: limit lower=0.0 upper=0.0 effort=1.0 velocity=0.0 -> lower=0.0 upper=0.0 effort=10.0 velocity=0.0; origin xyz=0 -0.16496 -0.30899 rpy=1.49669  0 1.57079 -> xyz=0 -0.16496 -0.30899 rpy=1.6 0 1.57079
- joint body_rocker_right: limit lower=0.0 upper=0.0 effort=1.0 velocity=0.0 -> lower=0.0 upper=0.0 effort=10.0 velocity=0.0; origin xyz=0       0.1649  -0.30899 rpy=1.57079 -0.0741   0 -> xyz=0       0.1649  -0.30899 rpy=1.57079 0 0
- joint bogie_left_corner_lf: limit lower=0.0 upper=0.0 effort=1.0 velocity=0.5 -> lower=0.0 upper=0.0 effort=10.0 velocity=0.5
- joint bogie_left_wheel_lm: limit lower=0.0 upper=0.0 effort=1.0 velocity=0.0 -> lower=0.0 upper=0.0 effort=10.0 velocity=0.0; origin xyz=0 0 0 rpy=0  0  0 -> xyz=0.10451 -0.17908  0.07827 rpy=0  0  0; parent wheel_lm_local -> bogie_left
- joint bogie_right_corner_rf: limit lower=0.0 upper=0.0 effort=1.0 velocity=0.5 -> lower=0.0 upper=0.0 effort=10.0 velocity=0.5
- joint bogie_right_wheel_rm: limit lower=0.0 upper=0.0 effort=1.0 velocity=0.0 -> lower=0.0 upper=0.0 effort=10.0 velocity=0.0; origin xyz=0 0 0 rpy=0  0  0 -> xyz=0.06634 -0.18198 -0.07859 rpy=0  0  0; parent wheel_rm_local -> bogie_right
- joint corner_lb_wheel_lb: limit lower=0.0 upper=0.0 effort=1.0 velocity=0.0 -> lower=0.0 upper=0.0 effort=10.0 velocity=0.0; origin xyz=0 0 0 rpy=0  0  0 -> xyz=0.04037 -0.06867  0.00497 rpy=0  0  0; parent wheel_lb_local -> corner_lb
- joint corner_lf_wheel_lf: limit lower=0.0 upper=0.0 effort=1.0 velocity=0.0 -> lower=0.0 upper=0.0 effort=10.0 velocity=0.0; origin xyz=0 0 0 rpy=0  0  0 -> xyz=0.02792 -0.08943  0.01005 rpy=0  0  0; parent wheel_lf_local -> corner_lf
- joint corner_rb_wheel_rb: limit lower=0.0 upper=0.0 effort=1.0 velocity=0.0 -> lower=0.0 upper=0.0 effort=10.0 velocity=0.0; origin xyz=0 0 0 rpy=0  0  0 -> xyz=0.0076  -0.09914 -0.01061 rpy=0  0  0; parent wheel_rb_local -> corner_rb
- joint corner_rf_wheel_rf: limit lower=0.0 upper=0.0 effort=1.0 velocity=0.0 -> lower=0.0 upper=0.0 effort=10.0 velocity=0.0; origin xyz=0 0 0 rpy=0  0  0 -> xyz=0.00407 -0.10082 -0.01036 rpy=0  0  0; parent wheel_rf_local -> corner_rf
- joint rocker_left_bogie_left: limit lower=0.0 upper=0.0 effort=1.0 velocity=0.0 -> lower=0.0 upper=0.0 effort=10.0 velocity=0.0
- joint rocker_left_corner_lb: limit lower=0.0 upper=0.0 effort=1.0 velocity=0.5 -> lower=0.0 upper=0.0 effort=10.0 velocity=0.5
- joint rocker_right_bogie_right: limit lower=0.0 upper=0.0 effort=1.0 velocity=0.0 -> lower=0.0 upper=0.0 effort=10.0 velocity=0.0
- joint rocker_right_corner_rb: limit lower=0.0 upper=0.0 effort=1.0 velocity=0.5 -> lower=0.0 upper=0.0 effort=10.0 velocity=0.5

File: src/khm_description/urdf/khm_description.urdf (robot description, URDF)
Before this commit: robot khm_description, 26 links, 25 joints
Links:
- removed link camera_link
- removed link depthcamera_link
- removed link imu_link
- removed link pointcloud_link
- added link front_imu_rocker_left
- added link front_imu_rocker_right
- added link wheel_lf_thermal_frame
Joints:
- removed joint camera_joint
- removed joint depthcamera_joint
- removed joint imu_joint
- removed joint pointcloud_joint
- added joint corner_lf_wheel_lf_thermal_frame: type fixed, parent corner_lf, child wheel_lf_thermal_frame, origin xyz=0.0 0.0 0.0 rpy=1.575 0.000 3.067
- added joint rocker_left_front_imu: type fixed, parent rocker_left, child front_imu_rocker_left, origin xyz=0 0 0 rpy=0 1.507 0
- added joint rocker_right_front_imu: type fixed, parent rocker_right, child front_imu_rocker_right, origin xyz=0 0 0 rpy=0 3.14 0
- joint body_rocker_left: limit lower=0.0 upper=0.0 effort=1.0 velocity=0.0 -> lower=0.0 upper=0.0 effort=10.0 velocity=0.0; origin xyz=0 -0.16496 -0.30899 rpy=1.49669  0 1.57079 -> xyz=0 -0.16496 -0.30899 rpy=1.6 0 1.57079
- joint body_rocker_right: limit lower=0.0 upper=0.0 effort=1.0 velocity=0.0 -> lower=0.0 upper=0.0 effort=10.0 velocity=0.0; origin xyz=0       0.1649  -0.30899 rpy=1.57079 -0.0741   0 -> xyz=0       0.1649  -0.30899 rpy=1.57079 0 0
- joint bogie_left_corner_lf: limit lower=0.0 upper=0.0 effort=1.0 velocity=0.5 -> lower=0.0 upper=0.0 effort=10.0 velocity=0.5
- joint bogie_left_wheel_lm: limit lower=0.0 upper=0.0 effort=1.0 velocity=0.0 -> lower=0.0 upper=0.0 effort=10.0 velocity=0.0
- joint bogie_right_corner_rf: limit lower=0.0 upper=0.0 effort=1.0 velocity=0.5 -> lower=0.0 upper=0.0 effort=10.0 velocity=0.5
- joint bogie_right_wheel_rm: limit lower=0.0 upper=0.0 effort=1.0 velocity=0.0 -> lower=0.0 upper=0.0 effort=10.0 velocity=0.0
- joint corner_lb_wheel_lb: limit lower=0.0 upper=0.0 effort=1.0 velocity=0.0 -> lower=0.0 upper=0.0 effort=10.0 velocity=0.0
- joint corner_lf_wheel_lf: limit lower=0.0 upper=0.0 effort=1.0 velocity=0.0 -> lower=0.0 upper=0.0 effort=10.0 velocity=0.0
- joint corner_rb_wheel_rb: limit lower=0.0 upper=0.0 effort=1.0 velocity=0.0 -> lower=0.0 upper=0.0 effort=10.0 velocity=0.0
- joint corner_rf_wheel_rf: limit lower=0.0 upper=0.0 effort=1.0 velocity=0.0 -> lower=0.0 upper=0.0 effort=10.0 velocity=0.0
- joint rocker_left_bogie_left: limit lower=0.0 upper=0.0 effort=1.0 velocity=0.0 -> lower=0.0 upper=0.0 effort=10.0 velocity=0.0
- joint rocker_left_corner_lb: limit lower=0.0 upper=0.0 effort=1.0 velocity=0.5 -> lower=0.0 upper=0.0 effort=10.0 velocity=0.5
- joint rocker_right_bogie_right: limit lower=0.0 upper=0.0 effort=1.0 velocity=0.0 -> lower=0.0 upper=0.0 effort=10.0 velocity=0.0
- joint rocker_right_corner_rb: limit lower=0.0 upper=0.0 effort=1.0 velocity=0.5 -> lower=0.0 upper=0.0 effort=10.0 velocity=0.5
- joint root_to_body: origin xyz=0 0 0 rpy=0 0 0 -> xyz=0 0 0 rpy=0 0 3.14159
