Commit message: visual updates

File: src/khm_description/urdf/khm_description.urdf (robot description, URDF)
Before this commit: robot khm_description, 26 links, 25 joints
Links:
- removed link base_scan
- added link rover_root
Joints:
- removed joint scan_joint
- added joint root_to_body: type fixed, parent rover_root, child body, origin xyz=0 0 0 rpy=0 0 0

Commit message: dev

File: src/khm_description/urdf/khm_description.urdf (robot description, URDF)
Before this commit: robot khm_description, 26 links, 25 joints
Links:
- link wheel_lb: geometry collision mesh filename=package://khm_description/meshes/wheel_lb_col.STL scale=1 1 1; visual mesh filename=package://khm_description/meshes/wheel_lb.dae scale=1 1 1
- link wheel_lf: geometry collision mesh filename=package://khm_description/meshes/wheel_lf_col.STL scale=1 1 1; visual mesh filename=package://khm_description/meshes/wheel_lf.dae scale=1 1 1
- link wheel_lm: geometry collision mesh filename=package://khm_description/meshes/wheel_lm_col.STL scale=1 1 1; visual mesh filename=package://khm_description/meshes/wheel_lm.dae scale=1 1 1
- link wheel_rb: geometry collision mesh filename=package://khm_description/meshes/wheel_rb_col.STL scale=1 1 1; visual mesh filename=package://khm_description/meshes/wheel_rb.dae scale=1 1 1
- link wheel_rf: geometry collision mesh filename=package://khm_description/meshes/wheel_rf_col.STL scale=1 1 1; visual mesh filename=package://khm_description/meshes/wheel_rf.dae scale=1 1 1
- link wheel_rm: geometry collision mesh filename=package://khm_description/meshes/wheel_rm_col.STL scale=1 1 1; visual mesh filename=package://khm_description/meshes/wheel_rm.dae scale=1 1 1

File: src/khm_description/urdf/khm_no_sensors_description.urdf (robot description, URDF)
Before this commit: robot khm_description, 22 links, 21 joints
Links:
- added link depthcamera_link
- added link wheel_lf_thermal_frame
- link wheel_lb: geometry collision mesh filename=package://khm_description/meshes/wheel_lb_col.STL scale=1 1 1; visual mesh filename=package://khm_description/meshes/wheel_lb.dae scale=1 1 1
- link wheel_lf: geometry collision mesh filename=package://khm_description/meshes/wheel_lf_col.STL scale=1 1 1; visual mesh filename=package://khm_description/meshes/wheel_lf.dae scale=1 1 1
- link wheel_lm: geometry collision mesh filename=package://khm_description/meshes/wheel_lm_col.STL scale=1 1 1; visual mesh filename=package://khm_description/meshes/wheel_lm.dae scale=1 1 1
- link wheel_rb: geometry collision mesh filename=package://khm_description/meshes/wheel_rb_col.STL scale=1 1 1; visual mesh filename=package://khm_description/meshes/wheel_rb.dae scale=1 1 1
- link wheel_rf: geometry collision mesh filename=package://khm_description/meshes/wheel_rf_col.STL scale=1 1 1; visual mesh filename=package://khm_description/meshes/wheel_rf.dae scale=1 1 1
- link wheel_rm: geometry collision mesh filename=package://khm_description/meshes/wheel_rm_col.STL scale=1 1 1; visual mesh filename=package://khm_description/meshes/wheel_rm.dae scale=1 1 1
Joints:
- added joint corner_lf_wheel_lf_thermal_frame: type fixed, parent corner_lf, child wheel_lf_thermal_frame, origin xyz=0.0 0.0 0.0 rpy=1.575 0.000 3.067
- added joint root_to_depthcamera: type fixed, parent rover_root, child depthcamera_link, origin xyz=0.1 0 -0.2 rpy=0 0 0
- joint root_to_body: origin xyz=0 0 0 rpy=0 0 0 -> xyz=0 0 0 rpy=0 0 3.14159

Commit message: add new wheels

File: src/khm_description/urdf/khm_description.urdf (robot description, URDF)
Before this commit: robot khm_description, 25 links, 24 joints
Links:
- link wheel_lb: geometry collision mesh filename=package://khm_description/meshes/simple_wheel_col.STL scale=1 1 1; visual mesh filename=package://khm_description/meshes/wheel_lb.dae scale=1 1 1
- link wheel_lf: geometry collision mesh filename=package://khm_description/meshes/simple_wheel_col.STL scale=1 1 1; visual mesh filename=package://khm_description/meshes/wheel_lf.dae scale=1 1 1
- link wheel_lm: geometry collision mesh filename=package://khm_description/meshes/simple_wheel_col.STL scale=1 1 1; visual mesh filename=package://khm_description/meshes/wheel_lm.dae scale=1 1 1
- link wheel_rb: geometry collision mesh filename=package://khm_description/meshes/simple_wheel_col.STL scale=1 1 1; visual mesh filename=package://khm_description/meshes/wheel_rb.dae scale=1 1 1
- link wheel_rf: geometry collision mesh filename=package://khm_description/meshes/simple_wheel_col.STL scale=1 1 1; visual mesh filename=package://khm_description/meshes/wheel_rf.dae scale=1 1 1
- link wheel_rm: geometry collision mesh filename=package://khm_description/meshes/simple_wheel_col.STL scale=1 1 1; visual mesh filename=package://khm_description/meshes/wheel_rm.dae scale=1 1 1

Commit message: revert wheels back (custom wheels buggy)

File: src/khm_description/urdf/khm_description.urdf (robot description, URDF)
Before this commit: robot khm_description, 25 links, 24 joints
Links:
- link wheel_lb: geometry collision mesh filename=package://khm_description/meshes/wheel_col.STL scale=1 1 1; visual mesh filename=package://khm_description/meshes/wheel_lb.dae scale=1 1 1
- link wheel_lf: geometry collision mesh filename=package://khm_description/meshes/wheel_col.STL scale=1 1 1; visual mesh filename=package://khm_description/meshes/wheel_lf.dae scale=1 1 1
- link wheel_lm: geometry collision mesh filename=package://khm_description/meshes/wheel_col.STL scale=1 1 1; visual mesh filename=package://khm_description/meshes/wheel_lm.dae scale=1 1 1
- link wheel_rb: geometry collision mesh filename=package://khm_description/meshes/wheel_col.STL scale=1 1 1; visual mesh filename=package://khm_description/meshes/wheel_rb.dae scale=1 1 1
- link wheel_rf: geometry collision mesh filename=package://khm_description/meshes/wheel_col.STL scale=1 1 1; visual mesh filename=package://khm_description/meshes/wheel_rf.dae scale=1 1 1
- link wheel_rm: geometry collision mesh filename=package://khm_description/meshes/wheel_col.STL scale=1 1 1; visual mesh filename=package://khm_description/meshes/wheel_rm.dae scale=1 1 1

File: src/khm_description/urdf/khm_no_sensors_description.urdf (robot description, URDF)
Before this commit: robot khm_description, 23 links, 22 joints
Links:
- link wheel_lb: geometry collision mesh filename=package://khm_description/meshes/wheel_col.STL scale=1 1 1; visual mesh filename=package://khm_description/meshes/wheel_lb.dae scale=1 1 1
- link wheel_lf: geometry collision mesh filename=package://khm_description/meshes/wheel_col.STL scale=1 1 1; visual mesh filename=package://khm_description/meshes/wheel_lf.dae scale=1 1 1
- link wheel_lm: geometry collision mesh filename=package://khm_description/meshes/wheel_col.STL scale=1 1 1; visual mesh filename=package://khm_description/meshes/wheel_lm.dae scale=1 1 1
- link wheel_rb: geometry collision mesh filename=package://khm_description/meshes/wheel_col.STL scale=1 1 1; visual mesh filename=package://khm_description/meshes/wheel_rb.dae scale=1 1 1
- link wheel_rf: geometry collision mesh filename=package://khm_description/meshes/wheel_col.STL scale=1 1 1; visual mesh filename=package://khm_description/meshes/wheel_rf.dae scale=1 1 1
- link wheel_rm: geometry collision mesh filename=package://khm_description/meshes/wheel_col.STL scale=1 1 1; visual mesh filename=package://khm_description/meshes/wheel_rm.dae scale=1 1 1
